File: 05-Layout/nowae021/nowae021-0/nowae021.kicad_pcb (KiCad board)
At the start: 2 copper layers, 21.6 x 20.3 mm, 39 parts, among them P1 NVT_BUS, P2 NVT_BUS, P3 SWD, Q1 PDTC123EU, Q2 PDTC123EU, Q3 PDTC123EU, Q4 PDTC123EU, Q5 PDTC123EU, Q6 PDTC123EU, SW1 BUTTON-WE_434153017835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

Commit message: Added license logos
Parts:
- added G***: LOGO, EXTLOGO:LOGO_OSH_5MM_FSILK, F.Cu at (120.5, 87.5)
- added G***: LOGO, EXTLOGO:LOGO_CC-BY-SA_5MM_FSILK, F.Cu at (120.4, 72.7)
- moved G*** 0.36 mm to (116.7, 79.5)
Other:
- board text added: "NOWAE021-0"
